File: Shared/laser-project/schematics/full-board-schematic/full-board-rev-a.sch (KiCad schematic (older format))
At the start: 44 parts, among them CON1 USB-B, SW1 PUSHSWITCH, T1 OP598C, T2 BSS138, T3 BSS138, U1 AT90USB1286, U2 DS1077, U3 AD8302, U4 MCP1825, U5 MCP1825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

Commit message: Finalized schematic.
Parts:
- removed C11, C12, C13: SMCAP, ~, symbol SMCAP
- removed X1: CERAMIC-RESONATOR, ~, symbol CERAMIC-RESONATOR
- added C17: SMCAP, ~, symbol SMCAP
- added SW2: PUSHSWITCH, ~, symbol PUSHSWITCH
- added X1: CSTCE16M0, ~, symbol CSTCE16M0
- C3: Capacitance 5p -> 100p
- C4: Capacitance 5p -> 100n
- C5, C7: Capacitance 5p? -> 1n
- C6, C8: Capacitance 5p? -> 200p
- R10: Resistance 91k -> 90.9k
- R2, R3: Resistance 10k? -> 56
- R4: Resistance 10k? -> 0
- R6: Resistance 750k -> 200k
- R7: Resistance 68k -> 16k
Connections:
- net labels added: hwb_sig
- wire segments 198 -> 201
Other:
- note added: "C1,C2\nMay be left open."
- moved on the sheet: C1, C16, C2, C3, C4, C5, C6, C7, C8, C9, R1, R2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
