File: Shared/laser-project/schematics/full-board-schematic/full-board-rev-a.sch (KiCad schematic (older format))
At the start: 43 parts, among them CON1 USB-MINI-B, SW1 PUSHSWITCH, SW2 PUSHSWITCH, T1 OP598C, T2 BSS138, T3 BSS138, U1 AT90USB1286, U2 DS1077, U3 AD8302, U4 MCP1825, U5 MCP1825, U6 6DOF, X1 CSTCE16M0

Commit message: Various schematic cleanups.
Fixed one actual error -- the ad8302 is supposed to be powered by
ad8302_vpos, not directly by regulator_5V.  The only difference is a
0ohm resistor and some caps.

Much of the cleanup came about because I was trying to find why the
rat's nest view for the pcb layout showed the at90usb1286 gnd and vcc
pins connected.  They weren't, actually.  Instead, there were many
lines between pins on that side, and only the non-overalapping parts
of the lines were drawn by kicad (thanks, kicad!).  So, I spent about
4 hours hunting down something that didn't exist.
Connections:
- net labels removed: A0, A1, A2, A3, A4, A5, A6, A7, B0, B1, B2, B3, B4, B5, B6, B7, C2, C3, C4, C5, C6, C7, D2, D3, D4, D5, D6, D7, E0, E1, E4, E5, E6, E7, F2, F3, F4, F5, F6, F7, regulator_5v
- wire segments 201 -> 133
- no-connect marks 4 -> 45
Other:
- moved on the sheet: C1, C17, C2, C3, C4, C9, R1, R5, R8, R9, T1, U2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

Commit message: Had forgotten to replace some labels.
While debugging, I had moved some regulator_5V labels to see if they
were causing a problem.  They weren't, but I forgot to move them back.
Connections:
- wire segments 133 -> 128
Changed lines of the file:
@@
 Text Label 8550 1200 0    60   ~ 0
 osc_ctrl0
-Text Label 1400 800  0    60   ~ 0
+Text Label 1200 800  0    60   ~ 0
 usb_5V
-Text Label 1400 900  0    60   ~ 0
+Text Label 1200 900  0    60   ~ 0
 usb_d-
-Text Label 1400 1000 0    60   ~ 0
+Text Label 1200 1000 0    60   ~ 0
 usb_d+
 $Comp
@@
 	1    0    0    -1
 $EndComp
-Text Label 2250 3850 0    60   ~ 0
+Text Label 2250 4050 0    60   ~ 0
 regulator_5V
 $Comp
@@
 Text Label 850  6750 0    60   ~ 0
 regulator_3.3V
-Text Label 1750 6650 0    60   ~ 0
+Text Label 1750 6750 0    60   ~ 0
 regulator_5V
 Text Label 1950 7300 0    60   ~ 0
@@
 Text Label 2750 6750 0    60   ~ 0
 regulator_3.3V
-Text Label 3750 6650 0    60   ~ 0
+Text Label 3650 6750 0    60   ~ 0
 regulator_5V
 Text Label 3850 7300 0    60   ~ 0
@@
 	8700 5400 9550 5400
 Wire Wire Line
-	1200 800  1700 800
-Wire Wire Line
-	1200 900  1700 900
-Wire Wire Line
-	1200 1000 1700 1000
-Wire Wire Line
 	1200 1200 1300 1200
 Wire Wire Line
@@
 	1750 7000 1750 6750
 Wire Wire Line
-	1750 6750 2100 6750
-Wire Wire Line
 	1250 7000 1250 6750
 Wire Wire Line
@@
 	3650 7000 3650 6750
 Wire Wire Line
-	3650 6750 4000 6750
-Wire Wire Line
 	3150 7000 3150 6750

Commit message: Continued routing work.
I still need to add some encoder interface pins.
Parts:
- added CON2: JTAG-10MIL-HDR, ~, symbol JTAG-10MIL-HDR
Connections:
- net labels added: jtag_tck, jtag_tdi, jtag_tdo, jtag_tms
- no-connect marks 45 -> 41
Other:
- moved on the sheet: C9, U2
Changed lines of the file:
@@
 LIBS:IMU
 LIBS:murataosc
+LIBS:jtag-10mil-header
 LIBS:full-board-rev-a-cache
 EELAYER 27 0
@@
 Sheet 1 1
 Title "Laser Mapping Project"
-Date "9 nov 2013"
+Date "10 nov 2013"
 Rev "A"
 Comp "Laser Team"
@@
 L DS1077 U2
 U 1 1 526F0599
-P 8250 1100
-F 0 "U2" H 8000 1400 60  0000 C CNN
-F 1 "DS1077" H 8350 1400 60  0000 C CNN
-F 2 "" H 8250 1100 60  0001 C CNN
-F 3 "" H 8250 1100 60  0001 C CNN
-	1    8250 1100
+P 9600 3000
+F 0 "U2" H 9350 3300 60  0000 C CNN
+F 1 "DS1077" H 9700 3300 60  0000 C CNN
+F 2 "" H 9600 3000 60  0001 C CNN
+F 3 "" H 9600 3000 60  0001 C CNN
+	1    9600 3000
 	1    0    0    -1
 $EndComp
@@
 L GND #PWR07
 U 1 1 52718D27
-P 7800 1400
-F 0 "#PWR07" H 7800 1400 30  0001 C CNN
-F 1 "GND" H 7800 1330 30  0001 C CNN
-F 2 "" H 7800 1400 60  0001 C CNN
-F 3 "" H 7800 1400 60  0001 C CNN
-	1    7800 1400
+P 9150 3300
+F 0 "#PWR07" H 9150 3300 30  0001 C CNN
+F 1 "GND" H 9150 3230 30  0001 C CNN
+F 2 "" H 9150 3300 60  0001 C CNN
+F 3 "" H 9150 3300 60  0001 C CNN
+	1    9150 3300
 	1    0    0    -1
 $EndComp
@@
 Text Label 8200 3600 0    60   ~ 0
 mod_sig_1
-Text Label 7800 900  2    60   ~ 0
+Text Label 9150 2800 2    60   ~ 0
 mod_sig_1
 $Comp
@@
 Text Label 5600 1000 0    60   ~ 0
 twi_sda_5V
-Text Label 8550 900  0    60   ~ 0
+Text Label 9900 2800 0    60   ~ 0
 twi_scl_5V
-Text Label 8550 1000 0    60   ~ 0
+Text Label 9900 2900 0    60   ~ 0
 twi_sda_5V
-Text Label 7650 1100 2    60   ~ 0
+Text Label 9000 3000 2    60   ~ 0
 regulator_5V
 $Comp
 L SMCAP C9
 U 1 1 527427A7
-P 7600 1300
-F 0 "C9" V 7700 1400 60  0000 C CNN
-F 1 "SMCAP" H 7850 1350 60  0001 C CNN
-F 2 "" H 7600 1300 60  0001 C CNN
-F 3 "" H 7600 1300 60  0001 C CNN
-F 4 "0.01u" V 7600 1450 60  0000 C CNN "Capacitance"
-	1    7600 1300
-	0    -1   -1   0
-$EndComp
-Text Label 8550 1100 0    60   ~ 0
+P 8950 3200
+F 0 "C9" V 9050 3300 60  0000 C CNN
+F 1 "SMCAP" H 9200 3250 60  0001 C CNN
+F 2 "" H 8950 3200 60  0001 C CNN
+F 3 "" H 8950 3200 60  0001 C CNN
+F 4 "0.01u" V 8950 3350 60  0000 C CNN "Capacitance"
+	1    8950 3200
+	0    -1   -1   0
+$EndComp
+Text Label 9900 3000 0    60   ~ 0
 osc_ctrl1
-Text Label 8550 1200 0    60   ~ 0
+Text Label 9900 3100 0    60   ~ 0
 osc_ctrl0
 Text Label 1200 800  0    60   ~ 0
@@
 NoConn ~ 1200 1100
 Wire Wire Line
-	7800 1200 7800 1400
-Wire Wire Line
-	7650 1350 7800 1350
-Connection ~ 7800 1350
-Wire Wire Line
-	7650 1100 7800 1100
-NoConn ~ 7800 1000
-Wire Wire Line
-	7650 1350 7650 1300
-Wire Wire Line
-	7650 1150 7650 1100
+	9150 3100 9150 3300
+Wire Wire Line
+	9000 3250 9150 3250
+Connection ~ 9150 3250
+Wire Wire Line
+	9000 3000 9150 3000
+NoConn ~ 9150 2900
+Wire Wire Line
+	9000 3250 9000 3200
+Wire Wire Line
+	9000 3050 9000 3000
 Wire Wire Line
 	3350 1550 3350 1500
@@
 NoConn ~ 5600 5600
 NoConn ~ 5600 5700
-NoConn ~ 5600 5800
-NoConn ~ 5600 5900
-NoConn ~ 5600 6000
-NoConn ~ 5600 6100
 NoConn ~ 3500 2700
 Wire Wire Line
@@
 Wire Wire Line
 	9200 3700 9200 3600
+Text Label 5600 5800 0    60   ~ 0
+jtag_tck
+Text Label 5600 5900 0    60   ~ 0
+jtag_tms
+Text Label 5600 6000 0    60   ~ 0
+jtag_tdo
+Text Label 5600 6100 0    60   ~ 0
+jtag_tdi
+$Comp
+L JTAG-10MIL-HDR CON2
+U 1 1 527EE66C
+P 9900 1200
+F 0 "CON2" H 9950 700 60  0000 C CNN
+F 1 "JTAG-10MIL-HDR" H 9900 1300 60  0000 C CNN
+F 2 "~" H 9700 1400 60  0000 C CNN
+F 3 "~" H 9700 1400 60  0000 C CNN
+	1    9900 1200
+	-1   0    0    1
+$EndComp
+Text Label 9650 1150 2    60   ~ 0
+jtag_tck
+Text Label 9650 1050 2    60   ~ 0
+jtag_tms
+Text Label 9650 950  2    60   ~ 0
+jtag_tdi
+Text Label 9650 850  2    60   ~ 0
+jtag_tdo
 $EndSCHEMATC

Commit message: More routing progress.
Also mounted a teensy++2.0 to the board.
Parts:
- added CON3: ENCODER-10MIL-HEADER, ~, symbol ENCODER-10MIL-HEADER
- added U7: TEENSYPP2, MODULE, symbol TEENSYPP2
Connections:
- net labels added: encoder-interface-0, encoder-interface-1, encoder-interface-2, encoder-interface-3, teensy-gnd
- wire segments 128 -> 131
- no-connect marks 41 -> 37
Other:
- moved on the sheet: C1, C10, C14, C15, C16, C17, C2, C3, C4, C5, C6, C7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
