File: Shared/laser-project/schematics/full-board-schematic/full-board-rev-a1.sch (KiCad schematic (older format))
At the start: 38 parts, among them CON1 ENCODER-10MIL-HEADER, CON2 JTAG-10MIL-HDR, T1 BSS138, T2 BSS138, T3 OP598C, U1 TEENSYPP2, U2 MCP1825, U3 DS1077, U4 AD8302, U5 MCP1825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

Commit message: 
Other:
- moved on the sheet: C8, C9, R11
Changed lines of the file:
@@
-EESchema Schematic File Version 2
+EESchema Schematic File Version 2  date 11/13/2013 3:26:50 PM
 LIBS:power
 LIBS:at90usb1286
@@
 LIBS:jtag-10mil-header
 LIBS:encoder-10mil-header
-EELAYER 27 0
+LIBS:buffer
+LIBS:full-board-rev-a1-cache
+EELAYER 24 0
 EELAYER END
 $Descr USLetter 11000 8500
@@
 Sheet 1 1
 Title "Laser Mapping Project"
-Date "12 nov 2013"
+Date "13 nov 2013"
 Rev "A"
 Comp "Laser Team"
@@
 L GND #PWR02
 U 1 1 52718763
-P 7050 6550
-F 0 "#PWR02" H 7050 6550 30  0001 C CNN
-F 1 "GND" H 7050 6480 30  0001 C CNN
-F 2 "" H 7050 6550 60  0001 C CNN
-F 3 "" H 7050 6550 60  0001 C CNN
-	1    7050 6550
+P 7650 7000
+F 0 "#PWR02" H 7650 7000 30  0001 C CNN
+F 1 "GND" H 7650 6930 30  0001 C CNN
+F 2 "" H 7650 7000 60  0001 C CNN
+F 3 "" H 7650 7000 60  0001 C CNN
+	1    7650 7000
 	1    0    0    -1
 $EndComp
@@
 L GND #PWR03
 U 1 1 52718769
-P 7450 6550
-F 0 "#PWR03" H 7450 6550 30  0001 C CNN
-F 1 "GND" H 7450 6480 30  0001 C CNN
-F 2 "" H 7450 6550 60  0001 C CNN
-F 3 "" H 7450 6550 60  0001 C CNN
-	1    7450 6550
+P 8050 7000
+F 0 "#PWR03" H 8050 7000 30  0001 C CNN
+F 1 "GND" H 8050 6930 30  0001 C CNN
+F 2 "" H 8050 7000 60  0001 C CNN
+F 3 "" H 8050 7000 60  0001 C CNN
+	1    8050 7000
 	1    0    0    -1
 $EndComp
@@
 L SMCAP C9
 U 1 1 52740D9C
-P 7400 6400
-F 0 "C9" V 7500 6500 60  0000 C CNN
-F 1 "SMCAP" H 7650 6450 60  0001 C CNN
-F 2 "SM1210" H 7400 6400 60  0001 C CNN
-F 3 "" H 7400 6400 60  0001 C CNN
-F 4 "100p" V 7400 6500 60  0000 C CNN "Capacitance"
-	1    7400 6400
+P 8000 6850
+F 0 "C9" V 8100 6950 60  0000 C CNN
+F 1 "SMCAP" H 8250 6900 60  0001 C CNN
+F 2 "SM1210" H 8000 6850 60  0001 C CNN
+F 3 "" H 8000 6850 60  0001 C CNN
+F 4 "100p" V 8000 6950 60  0000 C CNN "Capacitance"
+	1    8000 6850
 	0    -1   -1   0
 $EndComp
@@
 L SMCAP C8
 U 1 1 52740DAB
-P 7000 6400
-F 0 "C8" V 7150 6500 60  0000 C CNN
-F 1 "SMCAP" H 7250 6450 60  0001 C CNN
-F 2 "SM1210" H 7000 6400 60  0001 C CNN
-F 3 "" H 7000 6400 60  0001 C CNN
-F 4 "100n" V 7050 6500 60  0000 C CNN "Capacitance"
-	1    7000 6400
+P 7600 6850
+F 0 "C8" V 7750 6950 60  0000 C CNN
+F 1 "SMCAP" H 7850 6900 60  0001 C CNN
+F 2 "SM1210" H 7600 6850 60  0001 C CNN
+F 3 "" H 7600 6850 60  0001 C CNN
+F 4 "100n" V 7650 6950 60  0000 C CNN "Capacitance"
+	1    7600 6850
 	0    -1   -1   0
 $EndComp
@@
 L SMRES R11
 U 1 1 52740E3B
-P 7400 6050
-F 0 "R11" V 7600 5850 60  0000 C CNN
-F 1 "SMRES" H 7700 6100 60  0001 C CNN
-F 2 "SM1210" H 7400 6050 60  0001 C CNN
-F 3 "" H 7400 6050 60  0001 C CNN
-F 4 "0" V 7500 5800 60  0000 C CNN "Resistance"
-	1    7400 6050
-	0    -1   -1   0
-$EndComp
-Text Label 7450 5700 0    60   ~ 0
+P 8000 6500
+F 0 "R11" V 8200 6300 60  0000 C CNN
+F 1 "SMRES" H 8300 6550 60  0001 C CNN
+F 2 "SM1210" H 8000 6500 60  0001 C CNN
+F 3 "" H 8000 6500 60  0001 C CNN
+F 4 "0" V 8100 6250 60  0000 C CNN "Resistance"
+	1    8000 6500
+	0    -1   -1   0
+$EndComp
+Text Label 8050 6150 0    60   ~ 0
 regulator_5V
-Text Label 7450 6200 0    60   ~ 0
+Text Label 8050 6650 0    60   ~ 0
 ad8302_vpos
 $Comp
@@
 Wire Wire Line
 	9850 4050 8750 4050
-Connection ~ 7450 5700
-Wire Wire Line
-	7450 6400 7450 6550
+Connection ~ 8050 6150
+Wire Wire Line
+	8050 6850 8050 7000
 Wire Wire Line
 	3850 5550 3850 5450
@@
 	1800 7150 1800 6900
 Wire Wire Line
-	1300 7150 1300 6900
+	1300 6900 1300 7150
 Wire Wire Line
 	1300 6900 900  6900
@@
 	4300 7200 4300 6950
 Wire Wire Line
-	3800 7200 3800 6950
+	3800 6950 3800 7200
 Wire Wire Line
 	3800 6950 3400 6950
@@
 Connection ~ 8950 1300
 Wire Wire Line
-	7450 5700 7450 5800
-Wire Wire Line
-	7450 6050 7450 6250
-Wire Wire Line
-	7050 6550 7050 6400
-Wire Wire Line
-	7050 6250 7050 5700
-Wire Wire Line
-	7050 5700 7450 5700
+	8050 6150 8050 6250
+Wire Wire Line
+	8050 6500 8050 6700
+Wire Wire Line
+	7650 7000 7650 6850
+Wire Wire Line
+	7650 6700 7650 6150
+Wire Wire Line
+	7650 6150 8050 6150
 Text Label 7900 4050 2    60   ~ 0
 ad8302_vpos

Commit message: 
Connections:
- net labels added: teensy_5V
- net labels removed: usb_5V
Changed lines of the file:
@@
-EESchema Schematic File Version 2  date 11/13/2013 3:26:50 PM
+EESchema Schematic File Version 2  date 11/13/2013 7:10:31 PM
 LIBS:power
 LIBS:at90usb1286
@@
 Sheet 1 1
 Title "Laser Mapping Project"
-Date "13 nov 2013"
+Date "14 nov 2013"
 Rev "A"
 Comp "Laser Team"
@@
 osc_ctrl0
 Text Label 7650 1300 0    60   ~ 0
-usb_5V
+teensy_5V
 $Comp
 L GND #PWR011
@@
 $EndComp
 Text Label 4950 1300 0    60   ~ 0
-usb_5V
+teensy_5V
 $Comp
 L GND #PWR014
@@
 $EndComp
 Text Label 3850 1400 0    40   ~ 0
-regulator_5V
+teensy_5V
 Text Label 3850 2500 0    40   ~ 0
 ad8302_vref

Commit message: Addition of the op-amp, ground planes, and milling finalization.
Parts:
- added U7: TI-OPA2356, ~, symbol TI-OPA2356
Connections:
- net labels added: laser_drive_sig
- wire segments 102 -> 107
- no-connect marks 3 -> 6
Changed lines of the file:
@@
-EESchema Schematic File Version 2  date 11/13/2013 7:10:31 PM
+EESchema Schematic File Version 2
 LIBS:power
 LIBS:at90usb1286
@@
 LIBS:encoder-10mil-header
 LIBS:buffer
-LIBS:full-board-rev-a1-cache
-EELAYER 24 0
+LIBS:ti-opa2356
+EELAYER 27 0
 EELAYER END
 $Descr USLetter 11000 8500
@@
 $EndComp
 Text Label 4550 3950 0    60   ~ 0
-mod_sig_1
+laser_drive_sig
 Text Label 5500 2750 2    60   ~ 0
 mod_sig_1
@@
 Text Label 3850 2700 0    40   ~ 0
 ad8302_phs
+Text Label 6750 5350 0    60   ~ 0
+regulator_5V
+$Comp
+L GND #PWR?
+U 1 1 528552A0
+P 5700 5800
+F 0 "#PWR?" H 5700 5800 30  0001 C CNN
+F 1 "GND" H 5700 5730 30  0001 C CNN
+F 2 "" H 5700 5800 60  0001 C CNN
+F 3 "" H 5700 5800 60  0001 C CNN
+	1    5700 5800
+	1    0    0    -1
+$EndComp
+Wire Wire Line
+	5700 5800 5700 5650
+Wire Wire Line
+	5700 5650 5800 5650
+Text Label 5800 5550 2    60   ~ 0
+mod_sig_1
+Wire Wire Line
+	5800 5350 5700 5350
+Wire Wire Line
+	5700 5350 5700 5450
+Wire Wire Line
+	5700 5450 5800 5450
+Text Label 5700 5350 2    60   ~ 0
+laser_drive_sig
+$Comp
+L TI-OPA2356 U7
+U 1 1 52855541
+P 5900 5250
+F 0 "U7" H 5950 5400 60  0000 C CNN
+F 1 "TI-OPA2356" H 6200 5300 60  0000 C CNN
+F 2 "~" H 5900 5050 60  0000 C CNN
+F 3 "~" H 5900 5050 60  0000 C CNN
+	1    5900 5250
+	1    0    0    -1
+$EndComp
+NoConn ~ 6750 5450
+NoConn ~ 6750 5550
+NoConn ~ 6750 5650
 $EndSCHEMATC
